File: SoundX.sch (KiCad schematic (older format))
At the start: 51 parts, among them CN1 EDGE_CONN, CN2 RAW_AUDIO_OUT, CN3 CONN_MIDI_IN, CN4 CONN_MIDI_OUT, U1 GAL20V8, U2 MOS_6551_ACIA, U3 YM3526, U4 6N138, U6 YM3014, U7 LM324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

Commit message: Add some P/Ns
Parts:
- C1, C15: MouserPN (none) -> 710-860010472002
- C12: MouserPN 810-FG28X7R1H104KNT0 -> (none)
- C13: MouserPN 810-FG28C0G1H471JNT6 -> (none)
- C5: MouserPN 710-860020573008 -> 710-860010472002
- C7: MouserPN (none) -> 810-FG28X7R1H104KNT0
- FB1, FB2, FB3: MouserPN 623-2743015112 -> 875-28C0236-0EW-10
- JP1, JP2, JP3, JP4, JP5: MouserPN (none) -> -
- U1: MouserPN (none) -> 556-AF22LV10CQZ-30PU
- U4: MouserPN (none) -> 859-6N138
- U7: MouserPN (none) -> 595-LM324N
- Y2: MouserPN (none) -> 520-HCA300-SX
Changed lines of the file:
@@
 F 3 "" H 13665 2585 50  0001 C CNN
 F 4 "COMMON" H 13665 2585 50  0001 C CNN "Notes"
+F 5 "556-AF22LV10CQZ-30PU" H 13665 2585 50  0001 C CNN "MouserPN"
 	1    13665 2585
 	1    0    0    -1
@@
 F 3 "~" H 1445 6945 50  0001 C CNN
 F 4 "OPL" H 1445 6945 50  0001 C CNN "Notes"
+F 5 "810-FG28X7R1H104KNT0" H 1445 6945 50  0001 C CNN "MouserPN"
 	1    1445 6945
 	1    0    0    -1
@@
 F 2 "Inductor_THT:L_Radial_D6.0mm_P4.00mm" V 3775 6945 50  0001 C CNN
 F 3 "~" H 3845 6945 50  0001 C CNN
-F 4 "623-2743015112" H 3845 6945 50  0001 C CNN "MouserPN"
+F 4 "875-28C0236-0EW-10" H 3845 6945 50  0001 C CNN "MouserPN"
 F 5 "OPL" H 3845 6945 50  0001 C CNN "Notes"
 	1    3845 6945
@@
 F 2 "Inductor_THT:L_Radial_D6.0mm_P4.00mm" V 2760 6230 50  0001 C CNN
 F 3 "~" H 2830 6230 50  0001 C CNN
-F 4 "623-2743015112" H 2830 6230 50  0001 C CNN "MouserPN"
+F 4 "875-28C0236-0EW-10" H 2830 6230 50  0001 C CNN "MouserPN"
 F 5 "OPL" H 2830 6230 50  0001 C CNN "Notes"
 	1    2830 6230
@@
 F 3 "~" H 2330 6935 50  0001 C CNN
 F 4 "OPL" H 2330 6935 50  0001 C CNN "Notes"
+F 5 "-" H 2330 6935 50  0001 C CNN "MouserPN"
 	1    2330 6935
 	0    -1   1    0
@@
 F 3 "http://www.ti.com/lit/ds/symlink/lm2902-n.pdf" H 9085 6470 50  0001 C CNN
 F 4 "OPL" H 9035 6270 50  0001 C CNN "Notes"
+F 5 "595-LM324N" H 9035 6270 50  0001 C CNN "MouserPN"
 	1    9035 6270
 	1    0    0    -1
@@
 F 3 "http://www.ti.com/lit/ds/symlink/lm2902-n.pdf" H 12635 5595 50  0001 C CNN
 F 4 "OPL" H 12585 5395 50  0001 C CNN "Notes"
+F 5 "595-LM324N" H 12585 5395 50  0001 C CNN "MouserPN"
 	2    12585 5395
 	1    0    0    1
@@
 F 3 "http://www.ti.com/lit/ds/symlink/lm2902-n.pdf" H 10950 6570 50  0001 C CNN
 F 4 "OPL" H 10900 6370 50  0001 C CNN "Notes"
+F 5 "595-LM324N" H 10900 6370 50  0001 C CNN "MouserPN"
 	3    10900 6370
 	1    0    0    -1
@@
 F 3 "http://www.ti.com/lit/ds/symlink/lm2902-n.pdf" H 11150 5495 50  0001 C CNN
 F 4 "OPL" H 11100 5295 50  0001 C CNN "Notes"
+F 5 "595-LM324N" H 11100 5295 50  0001 C CNN "MouserPN"
 	4    11100 5295
 	1    0    0    -1
@@
 F 3 "http://www.ti.com/lit/ds/symlink/lm2902-n.pdf" H 3640 10555 50  0001 C CNN
 F 4 "OPL" H 3590 10355 50  0001 C CNN "Notes"
+F 5 "595-LM324N" H 3590 10355 50  0001 C CNN "MouserPN"
 	5    3590 10355
 	1    0    0    -1
@@
 F 2 "Capacitor_THT:CP_Radial_D5.0mm_P2.00mm" H 10510 5445 50  0001 C CNN
 F 3 "~" H 10510 5445 50  0001 C CNN
-F 4 "710-860020573008" H 10510 5445 50  0001 C CNN "MouserPN"
+F 4 "710-860010472002" H 10510 5445 50  0001 C CNN "MouserPN"
 F 5 "OPL" H 10510 5445 50  0001 C CNN "Notes"
 	1    10510 5445
@@
 F 3 "~" H 13435 5395 50  0001 C CNN
 F 4 "OPL" H 13435 5395 50  0001 C CNN "Notes"
+F 5 "710-860010472002" H 13435 5395 50  0001 C CNN "MouserPN"
 	1    13435 5395
 	0    -1   -1   0
@@
 F 3 "~" H 13835 5595 50  0001 C CNN
 F 4 "OPL" H 13835 5595 50  0001 C CNN "Notes"
+F 5 "-" H 13835 5595 50  0001 C CNN "MouserPN"
 	1    13835 5595
 	1    0    0    -1
@@
 F 3 "~" H 12690 9080 50  0001 C CNN
 F 4 "MIDI" H 12690 9080 50  0001 C CNN "Notes"
+F 5 "-" H 12690 9080 50  0001 C CNN "MouserPN"
 	1    12690 9080
 	-1   0    0    1
@@
 F 3 "~" H 13405 8735 50  0001 C CNN
 F 4 "MIDI" H 13405 8735 50  0001 C CNN "Notes"
+F 5 "-" H 13405 8735 50  0001 C CNN "MouserPN"
 	1    13405 8735
 	-1   0    0    1
@@
 F 3 "http://www.onsemi.com/pub/Collateral/HCPL2731-D.pdf" H 8665 8705 50  0001 C CNN
 F 4 "MIDI" H 8375 9005 50  0001 C CNN "Notes"
+F 5 "859-6N138" H 8375 9005 50  0001 C CNN "MouserPN"
 	1    8375 9005
 	1    0    0    -1
@@
 F 3 "~" H 6380 1965 50  0001 C CNN
 F 4 "MIDI" H 6380 1965 50  0001 C CNN "Notes"
+F 5 "520-HCA300-SX" H 6380 1965 50  0001 C CNN "MouserPN"
 	1    6380 1965
 	0    -1   -1   0
@@
 F 2 "Capacitor_THT:C_Disc_D7.0mm_W2.5mm_P5.00mm" H 9983 6415 50  0001 C CNN
 F 3 "~" H 9945 6565 50  0001 C CNN
-F 4 "810-FG28C0G1H471JNT6" H 9945 6565 50  0001 C CNN "MouserPN"
+F 4 "" H 9945 6565 50  0001 C CNN "MouserPN"
 F 5 "OPL" H 9945 6565 50  0001 C CNN "Notes"
 	1    9945 6565
@@
 F 2 "Capacitor_THT:C_Disc_D7.0mm_W2.5mm_P5.00mm" H 6613 2290 50  0001 C CNN
 F 3 "~" H 6575 2440 50  0001 C CNN
-F 4 "810-FG28X7R1H104KNT0" H 6575 2440 50  0001 C CNN "MouserPN"
+F 4 "" H 6575 2440 50  0001 C CNN "MouserPN"
 F 5 "MIDI" H 6575 2440 50  0001 C CNN "Notes"
 	1    6575 2440
@@
 F 2 "Inductor_THT:L_Radial_D6.0mm_P4.00mm" V 1035 1060 50  0001 C CNN
 F 3 "~" H 1105 1060 50  0001 C CNN
-F 4 "623-2743015112" H 1105 1060 50  0001 C CNN "MouserPN"
+F 4 "875-28C0236-0EW-10" H 1105 1060 50  0001 C CNN "MouserPN"
 F 5 "COMMON" H 1105 1060 50  0001 C CNN "Notes"
 	1    1105 1060
@@
 F 3 "~" H 4015 10370 50  0001 C CNN
 F 4 "OPL" H 4015 10370 50  0001 C CNN "Notes"
+F 5 "710-860010472002" H 4015 10370 50  0001 C CNN "MouserPN"
 	1    4015 10370
 	1    0    0    -1
@@
 F 3 "~" H 11825 5950 50  0001 C CNN
 F 4 "OPL" H 11825 5950 50  0001 C CNN "Notes"
+F 5 "-" H 11825 5950 50  0001 C CNN "MouserPN"
 	1    11825 5950
 	-1   0    0    1
